File: 01_pcb/pcb.kicad_pcb (KiCad board)
At the start: 2 copper layers, 246.5 x 75 mm, 106 parts, among them J2 AVR-ISP-6_mod, J3 4PIN, J5 Conn_01x08, SW1 SW_PUSH, U1 ATmega32U4-A, Y1 16MHz

Commit message: centered the bottom row
Parts:
- removed D53, D57: D_Small, Diode_SMD:D_SOD-123
- removed MX53, MX57: MX-NoLED, marbastlib-mx:SW_MX_HS_1.25u
- MX26, MX39: footprint marbastlib-mx:SW_MX_HS_1u -> marbastlib-mx:SW_MX_HS_1.25u
- MX56: footprint marbastlib-mx:SW_MX_HS_1.25u -> marbastlib-mx:SW_MX_HS_1u
- moved D39 4.76 mm to (227.7, 107.7)
- moved D56 4.76 mm to (249.1, 107.7)
- moved MX56 4.76 mm to (241.7, 106.0)
- moved MX39 4.76 mm to (220.3, 106.0)
- moved J2 2.47 mm to (114.2, 105.9)
- moved RSW1 2.47 mm to (126.8, 105.8)
- moved SW1 2.47 mm to (133.3, 105.9)
- moved C1 2.38 mm to (164.2, 101.0)
- moved C2 2.38 mm to (164.2, 109.0)
- moved C3 2.38 mm to (180.4, 112.8)
- moved MX54 2.38 mm to (56.0, 106.0)
- moved C4 2.38 mm to (183.8, 98.7)
- moved C5 2.38 mm to (176.1, 92.0)
- moved CX1 2.38 mm to (190.4, 103.2)
- moved CX2 2.38 mm to (190.4, 105.9)
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Routing:
- net GND: track 234.7 -> 292.0 mm, vias 176 -> 227
- net row4: track 294.5 -> 254.7 mm, vias 6 -> 4
- net col7: track 90.3 -> 108.3 mm
- net mosi/col3: track 153.6 -> 146.4 mm
- net row3: track 356.1 -> 362.4 mm
- net col0: track 209.1 -> 203.0 mm
- net Net-(D57-A): track 5.73 -> 0.00 mm
- net Net-(D53-A): track 5.71 -> 0.00 mm
- net col1: track 192.2 -> 197.7 mm
- net VCC: track 285.9 -> 282.0 mm
- net sck/col2: track 189.2 -> 192.7 mm
- net row2: track 389.6 -> 393.0 mm
- net row1: track 402.4 -> 405.8 mm
- net col5: track 106.6 -> 109.8 mm
- net col6: track 65.4 -> 68.5 mm
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