File: 01_pcb/pcb.kicad_sch (KiCad schematic)
At the start: 106 parts, among them J2 AVR-ISP-6_mod, J3 4PIN, J5 Conn_01x08, SW1 SW_PUSH, U1 ATmega32U4-A, Y1 16MHz

Commit message: centered the bottom row
Parts:
- removed D53, D57: D_Small, Diode_SMD:D_SOD-123, symbol Device:D_Small
- removed MX53, MX57: MX-NoLED, marbastlib-mx:SW_MX_HS_1.25u, symbol MX_Alps_Hybrid:MX-NoLED
- MX26, MX39: footprint marbastlib-mx:SW_MX_HS_1u -> marbastlib-mx:SW_MX_HS_1.25u
- MX56: footprint marbastlib-mx:SW_MX_HS_1.25u -> marbastlib-mx:SW_MX_HS_1u
Changed lines of the file:
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@@
   (junction (at 190.5 81.28) (diameter 0) (color 0 0 0 0)
   )
-  (junction (at 214.63 128.27) (diameter 0) (color 0 0 0 0)
-  )
   (junction (at 121.92 254) (diameter 0) (color 0 0 0 0)
   )
@@
   (junction (at 115.57 91.44) (diameter 0) (color 0 0 0 0)
   )
-  (junction (at 49.53 128.27) (diameter 0) (color 0 0 0 0)
-  )
   (junction (at 132.08 259.08) (diameter 0) (color 0 0 0 0)
   )
@@
   (junction (at 157.48 81.28) (diameter 0) (color 0 0 0 0)
   )
-  (junction (at 58.42 99.06) (diameter 0) (color 0 0 0 0)
-  )
   (junction (at 214.63 73.66) (diameter 0) (color 0 0 0 0)
   )
@@
   (junction (at 76.2 162.56) (diameter 0) (color 0 0 0 0)
   )
-  (junction (at 240.03 99.06) (diameter 0) (color 0 0 0 0)
-  )
   (junction (at 223.52 99.06) (diameter 0) (color 0 0 0 0)
   )
@@
     (stroke (width 0) (type default))
   )
-  (wire (pts (xy 39.37 128.27) (xy 49.53 128.27))
+  (wire (pts (xy 39.37 128.27) (xy 66.04 128.27))
     (stroke (width 0) (type default))
   )
@@
     (stroke (width 0) (type default))
   )
-  (wire (pts (xy 58.42 99.06) (xy 58.42 118.11))
-    (stroke (width 0) (type default))
-  )
   (wire (pts (xy 148.59 104.14) (xy 151.13 104.14))
     (stroke (width 0) (type default))
@@
     (stroke (width 0) (type default))
   )
-  (wire (pts (xy 240.03 118.11) (xy 238.76 118.11))
-    (stroke (width 0) (type default))
-  )
   (wire (pts (xy 115.57 91.44) (xy 132.08 91.44))
     (stroke (width 0) (type default))
@@
     (stroke (width 0) (type default))
   )
-  (wire (pts (xy 214.63 128.27) (xy 231.14 128.27))
-    (stroke (width 0) (type default))
-  )
   (wire (pts (xy 165.1 73.66) (xy 181.61 73.66))
     (stroke (width 0) (type default))
@@
     (stroke (width 0) (type default))
   )
-  (wire (pts (xy 58.42 118.11) (xy 57.15 118.11))
-    (stroke (width 0) (type default))
-  )
   (wire (pts (xy 190.5 63.5) (xy 190.5 81.28))
     (stroke (width 0) (type default))
@@
     (stroke (width 0) (type default))
   )
-  (wire (pts (xy 240.03 99.06) (xy 240.03 118.11))
-    (stroke (width 0) (type default))
-  )
   (wire (pts (xy 58.42 81.28) (xy 58.42 99.06))
     (stroke (width 0) (type default))
@@
     (stroke (width 0) (type default))
   )
-  (wire (pts (xy 49.53 128.27) (xy 66.04 128.27))
-    (stroke (width 0) (type default))
-  )
   (wire (pts (xy 214.63 123.19) (xy 217.17 123.19))
     (stroke (width 0) (type default))
@@
     (stroke (width 0) (type default))
   )
-  (wire (pts (xy 49.53 123.19) (xy 52.07 123.19))
-    (stroke (width 0) (type default))
-  )
   (wire (pts (xy 175.26 247.65) (xy 175.26 248.92))
     (stroke (width 0) (type default))
@@
     (stroke (width 0) (type default))
   )
-  (wire (pts (xy 231.14 123.19) (xy 233.68 123.19))
-    (stroke (width 0) (type default))
-  )
   (wire (pts (xy 57.15 81.28) (xy 58.42 81.28))
     (stroke (width 0) (type default))
@@
     )
   )
-  (symbol (lib_id "Device:D_Small") (at 49.53 125.73 90) (unit 1)
-    (in_bom yes) (on_board yes) (dnp no)
-    (property "Reference" "D53" (at 47.498 127 90)
-      (effects (font (size 1.27 1.27)) (justify left))
-    )
-    (property "Value" "D_Small" (at 51.562 129.54 90)
-      (effects (font (size 1.27 1.27)) (justify left))
-    )
-    (property "Footprint" "Diode_SMD:D_SOD-123" (at 49.53 125.73 90)
-      (effects (font (size 1.27 1.27)) hide)
-    )
-    (property "Datasheet" "~" (at 49.53 125.73 90)
-      (effects (font (size 1.27 1.27)) hide)
-    )
-    (property "Sim.Device" "D" (at 49.53 125.73 0)
-      (effects (font (size 1.27 1.27)) hide)
-    )
-    (property "Sim.Pins" "1=K 2=A" (at 49.53 125.73 0)
-      (effects (font (size 1.27 1.27)) hide)
-    )
-    (pin "1")
-    (pin "2")
-    (instances
-      (project "pcb"
-        (path "/b194be25-3710-4c98-baf2-77bb15d5dc1d"
-          (reference "D53") (unit 1)
-        )
-      )
-      (project "pcb"
-        (path "/b5352a33-563a-4ffe-a231-2e68fb54afa3"
-          (reference "D49") (unit 1)
-        )
-      )
-    )
-  )
   (symbol (lib_id "Device:D_Small") (at 198.12 71.12 90) (unit 1)
     (in_bom yes) (on_board yes) (dnp no)
@@
     )
   )
-  (symbol (lib_id "MX_Alps_Hybrid:MX-NoLED") (at 53.34 119.38 0) (unit 1)
-    (in_bom yes) (on_board yes) (dnp no)
-    (property "Reference" "MX53" (at 52.705 115.57 0)
-      (effects (font (size 1.524 1.524)))
-    )
-    (property "Value" "MX-NoLED" (at 52.705 118.11 0)
-      (effects (font (size 0.508 0.508)))
-    )
-    (property "Footprint" "marbastlib-mx:SW_MX_HS_1.25u" (at 37.465 120.015 0)
-      (effects (font (size 1.524 1.524)) hide)
-    )
-    (property "Datasheet" "" (at 37.465 120.015 0)
-      (effects (font (size 1.524 1.524)) hide)
-    )
-    (pin "1")
-    (pin "2")
-    (instances
-      (project "pcb"
-        (path "/b194be25-3710-4c98-baf2-77bb15d5dc1d"
-          (reference "MX53") (unit 1)
-        )
-      )
-      (project "pcb"
-        (path "/b5352a33-563a-4ffe-a231-2e68fb54afa3"
-          (reference "MX49") (unit 1)
-        )
-      )
-    )
-  )
   (symbol (lib_id "Device:R") (at 59.69 195.58 90) (unit 1)
     (in_bom yes) (on_board yes) (dnp no)
@@
       (effects (font (size 0.508 0.508)))
     )
-    (property "Footprint" "marbastlib-mx:SW_MX_HS_1u" (at 186.055 120.015 0)
+    (property "Footprint" "marbastlib-mx:SW_MX_HS_1.25u" (at 186.055 120.015 0)
       (effects (font (size 1.524 1.524)) hide)
     )
@@
       (effects (font (size 0.508 0.508)))
     )
-    (property "Footprint" "marbastlib-mx:SW_MX_HS_1u" (at 70.485 120.015 0)
+    (property "Footprint" "marbastlib-mx:SW_MX_HS_1.25u" (at 70.485 120.015 0)
       (effects (font (size 1.524 1.524)) hide)
     )
@@
       (effects (font (size 0.508 0.508)))
     )
-    (property "Footprint" "marbastlib-mx:SW_MX_HS_1.25u" (at 202.565 120.015 0)
+    (property "Footprint" "marbastlib-mx:SW_MX_HS_1u" (at 202.565 120.015 0)
       (effects (font (size 1.524 1.524)) hide)
     )
@@
     )
   )
-  (symbol (lib_id "MX_Alps_Hybrid:MX-NoLED") (at 234.95 119.38 0) (unit 1)
-    (in_bom yes) (on_board yes) (dnp no)
-    (property "Reference" "MX57" (at 234.315 115.57 0)
-      (effects (font (size 1.524 1.524)))
-    )
-    (property "Value" "MX-NoLED" (at 234.315 118.11 0)
-      (effects (font (size 0.508 0.508)))
-    )
-    (property "Footprint" "marbastlib-mx:SW_MX_HS_1.25u" (at 219.075 120.015 0)
-      (effects (font (size 1.524 1.524)) hide)
-    )
-    (property "Datasheet" "" (at 219.075 120.015 0)
-      (effects (font (size 1.524 1.524)) hide)
-    )
-    (pin "1")
-    (pin "2")
-    (instances
-      (project "pcb"
-        (path "/b194be25-3710-4c98-baf2-77bb15d5dc1d"
-          (reference "MX57") (unit 1)
-        )
-      )
-      (project "pcb"
-        (path "/b5352a33-563a-4ffe-a231-2e68fb54afa3"
-          (reference "MX11") (unit 1)
-        )
-      )
-    )
-  )
   (symbol (lib_id "Device:D_Small") (at 181.61 71.12 90) (unit 1)
     (in_bom yes) (on_board yes) (dnp no)
@@
         )
       )
-    )
-  )
-  (symbol (lib_id "Device:D_Small") (at 231.14 125.73 90) (unit 1)
-    (in_bom yes) (on_board yes) (dnp no)
-    (property "Reference" "D57" (at 229.108 127 90)
-      (effects (font (size 1.27 1.27)) (justify left))
-    )
-    (property "Value" "D_Small" (at 233.172 129.54 90)
-      (effects (font (size 1.27 1.27)) (justify left))
-    )
-    (property "Footprint" "Diode_SMD:D_SOD-123" (at 231.14 125.73 90)
-      (effects (font (size 1.27 1.27)) hide)
-    )
-    (property "Datasheet" "~" (at 231.14 125.73 90)
-      (effects (font (size 1.27 1.27)) hide)
-    )
-    (property "Sim.Device" "D" (at 231.14 125.73 0)
-      (effects (font (size 1.27 1.27)) hide)
-    )
-    (property "Sim.Pins" "1=K 2=A" (at 231.14 125.73 0)
-      (effects (font (size 1.27 1.27)) hide)
-    )
-    (pin "1")
-    (pin "2")
-    (instances
-      (project "pcb"
-        (path "/b194be25-3710-4c98-baf2-77bb15d5dc1d"
-          (reference "D57") (unit 1)
-        )
-      )
-      (project "pcb"
-        (path "/b5352a33-563a-4ffe-a231-2e68fb54afa3"
-          (reference "D11") (unit 1)
-        )
-      )
